File: Hardware/Kicad/CPC_PICOROM_PLUS.kicad_sch (KiCad schematic)
At the start: 9 parts, among them J1 Amstrad_CPC_Plus_Expansion, SW1 Pico Reset, SW2 CPC Reset, U1 Pico

Commit message: 13-Dec-2024 updates
Parts:
- added JP1: Disable Internal ROMs, Jumper:SolderJumper-2_P1.3mm_Open_RoundedPad1.0x1.5mm, symbol Jumper:SolderJumper_2_Open
- J1: footprint CluelessEngineer:111050113L001 -> Clueless_Engineer:111050113L001_Amstrad_Plus
- SW1, SW2: footprint My_Components:Switch_Tactile_6mm -> Clueless_Engineer:Switch_Tactile_6mm
- U1: footprint CluelessEngineer:RPi_Pico_SMD_TH -> Clueless_Engineer:RPi_Pico_SMD_TH
Connections:
- net Vcc: now also JP1.2 (B); no longer J1.43 (ROMDIS)
- new net ROMDIS: J1.43 (ROMDIS), JP1.1 (A)
Other:
- moved on the sheet: SW1, SW2
